Commit message: 删除不必要的软件包，修改机器人的URDF

File: descriptions/at_dog_description/xacro/ros2_control_real.xacro (robot description, xacro)
@@ -5,5 +5,5 @@
 			<plugin>hardware_at_dog/HardwareATDog</plugin>
 		</hardware>
-		<joint name="lf_hip_joint">
+		<joint name="lf_joint1">
 			<command_interface name="position"/>
 			<command_interface name="velocity"/>
@@ -15,5 +15,5 @@
 			<state_interface name="effort"/>
 		</joint>
-		<joint name="lf_thigh_joint">
+		<joint name="lf_joint2">
 			<command_interface name="position"/>
 			<command_interface name="velocity"/>
@@ -25,5 +25,5 @@
 			<state_interface name="effort"/>
 		</joint>
-		<joint name="lf_calf_joint">
+		<joint name="lf_joint3">
 			<command_interface name="position"/>
 			<command_interface name="velocity"/>
@@ -35,5 +35,5 @@
 			<state_interface name="effort"/>
 		</joint>
-		<joint name="rf_hip_joint">
+		<joint name="rf_joint1">
 			<command_interface name="position"/>
 			<command_interface name="velocity"/>
@@ -45,5 +45,5 @@
 			<state_interface name="effort"/>
 		</joint>
-		<joint name="rf_thigh_joint">
+		<joint name="rf_joint2">
 			<command_interface name="position"/>
 			<command_interface name="velocity"/>
@@ -55,5 +55,5 @@
 			<state_interface name="effort"/>
 		</joint>
-		<joint name="rf_calf_joint">
+		<joint name="rf_joint3">
 			<command_interface name="position"/>
 			<command_interface name="velocity"/>
@@ -65,5 +65,5 @@
 			<state_interface name="effort"/>
 		</joint>
-		<joint name="lb_hip_joint">
+		<joint name="lb_joint1">
 			<command_interface name="position"/>
 			<command_interface name="velocity"/>
@@ -75,5 +75,5 @@
 			<state_interface name="effort"/>
 		</joint>
-		<joint name="lb_thigh_joint">
+		<joint name="lb_joint2">
 			<command_interface name="position"/>
 			<command_interface name="velocity"/>
@@ -85,5 +85,5 @@
 			<state_interface name="effort"/>
 		</joint>
-		<joint name="lb_calf_joint">
+		<joint name="lb_joint3">
 			<command_interface name="position"/>
 			<command_interface name="velocity"/>
@@ -95,5 +95,5 @@
 			<state_interface name="effort"/>
 		</joint>
-		<joint name="rb_hip_joint">
+		<joint name="rb_joint1">
 			<command_interface name="position"/>
 			<command_interface name="velocity"/>
@@ -105,5 +105,5 @@
 			<state_interface name="effort"/>
 		</joint>
-		<joint name="rb_thigh_joint">
+		<joint name="rb_joint2">
 			<command_interface name="position"/>
 			<command_interface name="velocity"/>
@@ -115,5 +115,5 @@
 			<state_interface name="effort"/>
 		</joint>
-		<joint name="rb_calf_joint">
+		<joint name="rb_joint3">
 			<command_interface name="position"/>
 			<command_interface name="velocity"/>
@@ -137,10 +137,4 @@
 			<state_interface name="linear_acceleration.z"/>
 		</sensor>
-		<sensor name="foot_force">
-			<state_interface name="lf"/>
-			<state_interface name="rf"/>
-			<state_interface name="lb"/>
-			<state_interface name="rb"/>
-		</sensor>
 		<sensor name="odometer">
 			<state_interface name="position.x"/>

File: descriptions/at_dog_description/xacro/ros2_control_sim.xacro (robot description, xacro)
@@ -93,10 +93,4 @@
 			<state_interface name="linear_acceleration.z"/>
 		</sensor>
-		<sensor name="foot_force">
-			<state_interface name="lf"/>
-			<state_interface name="rf"/>
-			<state_interface name="lb"/>
-			<state_interface name="rb"/>
-		</sensor>
 		<sensor name="odometer">
 			<state_interface name="position.x"/>

Commit message: 替换Mujoco硬件层接口软件包

File: descriptions/at_dog_description/xacro/ros2_control_real.xacro (robot description, xacro)
@@ -125,5 +125,5 @@
 			<state_interface name="effort"/>
 		</joint>
-		<sensor name="imu_sensor">
+		<sensor name="imu_main_imu">
 			<state_interface name="orientation.w"/>
 			<state_interface name="orientation.x"/>

File: descriptions/at_dog_description/xacro/ros2_control_sim.xacro (robot description, xacro)
@@ -1,104 +1,100 @@
 <?xml version="1.0"?>
 <robot xmlns:xacro="http://www.ros.org/wiki/xacro">
-	<ros2_control name="at_dog_sys" type="system">
-		<hardware>
+    <ros2_control name="at_dog_sys" type="system">
+        <hardware>
             <plugin>mujoco_ros2_control/MujocoSystem</plugin>
         </hardware>
-		<joint name="lf_joint1">
-			<command_interface name="effort"/>
-			<state_interface name="position"/>
-			<state_interface name="velocity"/>
-			<state_interface name="effort"/>
-		</joint>
-		<joint name="lf_joint2">
-			<command_interface name="effort"/>
-			<state_interface name="position"/>
-			<state_interface name="velocity"/>
-			<state_interface name="effort"/>
-		</joint>
-		<joint name="lf_joint3">
-			<command_interface name="effort"/>
-			<state_interface name="position"/>
-			<state_interface name="velocity"/>
-			<state_interface name="effort"/>
-		</joint>
-		<joint name="rf_joint1">
-			<command_interface name="effort"/>
-			<state_interface name="position"/>
-			<state_interface name="velocity"/>
-			<state_interface name="effort"/>
-		</joint>
-		<joint name="rf_joint2">
-			<command_interface name="effort"/>
-			<state_interface name="position"/>
-			<state_interface name="velocity"/>
-			<state_interface name="effort"/>
-		</joint>
-		<joint name="rf_joint3">
-			<command_interface name="effort"/>
-			<state_interface name="position"/>
-			<state_interface name="velocity"/>
-			<state_interface name="effort"/>
-		</joint>
-		<joint name="lb_joint1">
-			<command_interface name="effort"/>
-			<state_interface name="position"/>
-			<state_interface name="velocity"/>
-			<state_interface name="effort"/>
-		</joint>
-		<joint name="lb_joint2">
-			<command_interface name="effort"/>
-			<state_interface name="position"/>
-			<state_interface name="velocity"/>
-			<state_interface name="effort"/>
-		</joint>
-		<joint name="lb_joint3">
-			<command_interface name="effort"/>
-			<state_interface name="position"/>
-			<state_interface name="velocity"/>
-			<state_interface name="effort"/>
-		</joint>
-		<joint name="rb_joint1">
-			<command_interface name="effort"/>
-			<state_interface name="position"/>
-			<state_interface name="velocity"/>
-			<state_interface name="effort"/>
-		</joint>
-		<joint name="rb_joint2">
-			<command_interface name="effort"/>
-			<state_interface name="position"/>
-			<state_interface name="velocity"/>
-			<state_interface name="effort"/>
-		</joint>
-		<joint name="rb_joint3">
-			<command_interface name="position"/>
-			<command_interface name="velocity"/>
-			<command_interface name="effort"/>
-			<command_interface name="kp"/>
-			<command_interface name="kd"/>
-			<state_interface name="position"/>
-			<state_interface name="velocity"/>
-			<state_interface name="effort"/>
-		</joint>
-		<sensor name="imu_sensor">
-			<state_interface name="orientation.w"/>
-			<state_interface name="orientation.x"/>
-			<state_interface name="orientation.y"/>
-			<state_interface name="orientation.z"/>
-			<state_interface name="angular_velocity.x"/>
-			<state_interface name="angular_velocity.y"/>
-			<state_interface name="angular_velocity.z"/>
-			<state_interface name="linear_acceleration.x"/>
-			<state_interface name="linear_acceleration.y"/>
-			<state_interface name="linear_acceleration.z"/>
-		</sensor>
-		<sensor name="odometer">
-			<state_interface name="position.x"/>
-			<state_interface name="position.y"/>
-			<state_interface name="position.z"/>
-			<state_interface name="velocity.x"/>
-			<state_interface name="velocity.y"/>
-			<state_interface name="velocity.z"/>
-		</sensor>
-	</ros2_control>
+        <joint name="lf_joint1">
+            <command_interface name="effort" />
+            <state_interface name="position" />
+            <state_interface name="velocity" />
+            <state_interface name="effort" />
+        </joint>
+        <joint name="lf_joint2">
+            <command_interface name="effort" />
+            <state_interface name="position" />
+            <state_interface name="velocity" />
+            <state_interface name="effort" />
+        </joint>
+        <joint name="lf_joint3">
+            <command_interface name="effort" />
+            <state_interface name="position" />
+            <state_interface name="velocity" />
+            <state_interface name="effort" />
+        </joint>
+        <joint name="rf_joint1">
+            <command_interface name="effort" />
+            <state_interface name="position" />
+            <state_interface name="velocity" />
+            <state_interface name="effort" />
+        </joint>
+        <joint name="rf_joint2">
+            <command_interface name="effort" />
+            <state_interface name="position" />
+            <state_interface name="velocity" />
+            <state_interface name="effort" />
+        </joint>
+        <joint name="rf_joint3">
+            <command_interface name="effort" />
+            <state_interface name="position" />
+            <state_interface name="velocity" />
+            <state_interface name="effort" />
+        </joint>
+        <joint name="lb_joint1">
+            <command_interface name="effort" />
+            <state_interface name="position" />
+            <state_interface name="velocity" />
+            <state_interface name="effort" />
+        </joint>
+        <joint name="lb_joint2">
+            <command_interface name="effort" />
+            <state_interface name="position" />
+            <state_interface name="velocity" />
+            <state_interface name="effort" />
+        </joint>
+        <joint name="lb_joint3">
+            <command_interface name="effort" />
+            <state_interface name="position" />
+            <state_interface name="velocity" />
+            <state_interface name="effort" />
+        </joint>
+        <joint name="rb_joint1">
+            <command_interface name="effort" />
+            <state_interface name="position" />
+            <state_interface name="velocity" />
+            <state_interface name="effort" />
+        </joint>
+        <joint name="rb_joint2">
+            <command_interface name="effort" />
+            <state_interface name="position" />
+            <state_interface name="velocity" />
+            <state_interface name="effort" />
+        </joint>
+        <joint name="rb_joint3">
+            <command_interface name="effort" />
+            <state_interface name="position" />
+            <state_interface name="velocity" />
+            <state_interface name="effort" />
+        </joint>
+        <sensor name="imu_main_imu">
+            <state_interface name="orientation.w" />
+            <state_interface name="orientation.x" />
+            <state_interface name="orientation.y" />
+            <state_interface name="orientation.z" />
+            <state_interface name="angular_velocity.x" />
+            <state_interface name="angular_velocity.y" />
+            <state_interface name="angular_velocity.z" />
+            <state_interface name="linear_acceleration.x" />
+            <state_interface name="linear_acceleration.y" />
+            <state_interface name="linear_acceleration.z" />
+        </sensor>
+        <sensor name="odometer">
+            <state_interface name="position.x" />
+            <state_interface name="position.y" />
+            <state_interface name="position.z" />
+            <state_interface name="velocity.x" />
+            <state_interface name="velocity.y" />
+            <state_interface name="velocity.z" />
+        </sensor>
+    </ros2_control>
 </robot>
