Commit message: 使用了moveit__mujoco_ros2_control版本的桥接器，并修正了启动崩溃的问题

File: descriptions/at_dog_description/xacro/robot.xacro (robot description, xacro)
@@ -9,10 +9,10 @@
     <xacro:include filename="$(find at_dog_description)/xacro/ros2_control_real.xacro"/>
   </xacro:unless>
-  <!-- <joint name="imu_joint" type="fixed">
-    <parent link="trunk"/>
-    <child link="imu_link"/>
-    <origin rpy="0 0 0" xyz="0 0 0"/>
+  <joint name="imu_main_joint" type="fixed">
+    <parent link="body_link"/>
+    <child link="imu_main_link"/>
+    <origin rpy="0 0 0" xyz="0 0 0.056203"/>
   </joint>
-  <link name="imu_link">
+  <link name="imu_main_link">
     <inertial>
       <mass value="0.001"/>
@@ -33,4 +33,4 @@
       </geometry>
     </collision>
-  </link> -->
+  </link>
 </robot>

File: descriptions/at_dog_description/xacro/ros2_control_sim.xacro (robot description, xacro)
@@ -77,4 +77,16 @@
             <state_interface name="effort" />
         </joint>
+        <sensor name="imu_main_imu">
+            <state_interface name="orientation.x" />
+            <state_interface name="orientation.y" />
+            <state_interface name="orientation.z" />
+            <state_interface name="orientation.w" />
+            <state_interface name="angular_velocity.x" />
+            <state_interface name="angular_velocity.y" />
+            <state_interface name="angular_velocity.z" />
+            <state_interface name="linear_acceleration.x" />
+            <state_interface name="linear_acceleration.y" />
+            <state_interface name="linear_acceleration.z" />
+        </sensor>
     </ros2_control>
 </robot>
