Commit message: 仿真环境下的底层控制器配置完成

File: descriptions/at_dog_description/model/dog.urdf (robot description, URDF)
Before this commit: robot at_dog, 18 links, 17 joints
Links:
- removed link world
- link body_link: mass 3.1484 -> 4.2135; geometry collision mesh filename=package://at_dog_description/model/body_link.stl; visual mesh filename=package://at_dog_description/model/body_link.stl
- link lb_link1: mass 0.305258513351169 -> 0.305258519686429; geometry collision mesh filename=package://at_dog_description/model/lb_link1.stl; visual mesh filename=package://at_dog_description/model/lb_link1.stl
- link lb_link2: mass 0.682338727568128 -> 0.673603806804068; geometry collision mesh filename=package://at_dog_description/model/lb_link2.stl; visual mesh filename=package://at_dog_description/model/lb_link2.stl
- link lb_link3: mass 0.127541149243291 -> 0.119977441819341; geometry collision mesh filename=package://at_dog_description/model/lb_link3.stl; visual mesh filename=package://at_dog_description/model/lb_link3.stl
- link lb_link4: mass 0.65 -> 0.0781572031669603; geometry collision mesh filename=package://at_dog_description/model/lb_link4.stl; visual mesh filename=package://at_dog_description/model/lb_link4.stl
- link lf_link1: mass 0.30526 -> 0.305258503824178; geometry collision mesh filename=package://at_dog_description/model/lf_link1.stl; visual mesh filename=package://at_dog_description/model/lf_link1.stl
- link lf_link2: mass 0.687935058013005 -> 0.644661117972557; geometry collision mesh filename=package://at_dog_description/model/lf_link2.stl; visual mesh filename=package://at_dog_description/model/lf_link2.stl
- link lf_link3: mass 0.0715412570113012 -> 0.119977441819341; geometry collision mesh filename=package://at_dog_description/model/lf_link3.stl; visual mesh filename=package://at_dog_description/model/lf_link3.stl
- link lf_link4: mass 0.65 -> 0.0781571728156937; geometry collision mesh filename=package://at_dog_description/model/lf_link4.stl; visual mesh filename=package://at_dog_description/model/lf_link4.stl
- link rb_link1: mass 0.305258497916776 -> 0.305258557068333; geometry collision mesh filename=package://at_dog_description/model/rb_link1.stl; visual mesh filename=package://at_dog_description/model/rb_link1.stl
- link rb_link2: mass 0.682338712671127 -> 0.682338894787625; geometry collision mesh filename=package://at_dog_description/model/rb_link2.stl; visual mesh filename=package://at_dog_description/model/rb_link2.stl
- link rb_link3: mass 0.127541149243291 -> 0.119977441819341; geometry collision mesh filename=package://at_dog_description/model/rb_link3.stl; visual mesh filename=package://at_dog_description/model/rb_link3.stl
- link rb_link4: mass 0.65 -> 0.0781572323930169; geometry collision mesh filename=package://at_dog_description/model/rb_link4.stl; visual mesh filename=package://at_dog_description/model/rb_link4.stl
- link rf_link1: mass 0.305258520879218 -> 0.305258502432481; geometry collision mesh filename=package://at_dog_description/model/rf_link1.stl; visual mesh filename=package://at_dog_description/model/rf_link1.stl
- link rf_link2: mass 0.682338731946651 -> 0.65339621713157; geometry collision mesh filename=package://at_dog_description/model/rf_link2.stl; visual mesh filename=package://at_dog_description/model/rf_link2.stl
- link rf_link3: mass 0.127541149243291 -> 0.11997744181934; geometry collision mesh filename=package://at_dog_description/model/rf_link3.stl; visual mesh filename=package://at_dog_description/model/rf_link3.stl
- link rf_link4: mass 0.65 -> 0.0781571826488302; geometry collision mesh filename=package://at_dog_description/model/rf_link4.stl; visual mesh filename=package://at_dog_description/model/rf_link4.stl
Joints:
- removed joint float_joint
- joint lb_joint1: limit lower=-4 upper=4 effort=20 velocity=16 -> lower=-3 upper=3 effort=20 velocity=16
- joint lb_joint2: limit lower=-4 upper=4 effort=20 velocity=16 -> lower=-3 upper=3 effort=20 velocity=16; origin xyz=-0.00047387 -0.029283 0.059987 rpy=1.5708 0.0 0.0 -> xyz=7.0296E-05 -0.029287 0.059987 rpy=1.5708 0 0
- joint lb_joint3: limit lower=-4 upper=4 effort=20 velocity=16 -> lower=-3 upper=3 effort=20 velocity=16; origin xyz=0.23001 1.0811E-05 0.0935 rpy=0 0 -1.570796325 -> xyz=0.23001 0 0.0935 rpy=0 0 -1.5708
- joint lb_joint4: axis 0 0 1 -> 0 0 0; origin xyz=0.225 0 0.028 rpy=0 0 0 -> xyz=0.24313 0.012189 -0.023501 rpy=0 0 0
- joint lf_joint1: limit lower=-4 upper=4 effort=20 velocity=16 -> lower=-3 upper=3 effort=20 velocity=16
- joint lf_joint2: limit lower=-4 upper=4 effort=20 velocity=16 -> lower=-3 upper=3 effort=20 velocity=16; origin xyz=0 0.029313 0.060013 rpy=-1.5708 0.0 0 -> xyz=-0.000957 0.029298 0.060013 rpy=-1.5708 0 0
- joint lf_joint3: limit lower=-4 upper=4 effort=20 velocity=16 -> lower=-3 upper=3 effort=20 velocity=16; origin xyz=0.23001 0 0.0935 rpy=0 0 -1.570796325 -> xyz=0.23001 0 0.0935 rpy=0 0 -1.5708
- joint lf_joint4: axis 0 0 1 -> 0 0 0; origin xyz=0.225 0 0.028 rpy=0 0 0 -> xyz=0.243132280457965 0.0121889545734945 -0.0235007169194983 rpy=0 0 -3.14159265358976
- joint rb_joint1: limit lower=-4 upper=4 effort=20 velocity=16 -> lower=-3 upper=3 effort=20 velocity=16
- joint rb_joint2: limit lower=-4 upper=4 effort=20 velocity=16 -> lower=-3 upper=3 effort=20 velocity=16; origin xyz=-0.001301 0.029271 0.06 rpy=-1.5708 0 0 -> xyz=-0.0022402 0.029214 0.06 rpy=-1.5708 0 0
- joint rb_joint3: limit lower=-4 upper=4 effort=20 velocity=16 -> lower=-3 upper=3 effort=20 velocity=16; origin xyz=0.23 0 0.0935 rpy=0 0 1.570796325 -> xyz=0.23 0 0.0935 rpy=0 0 1.5708
- joint rb_joint4: axis 0 0 1 -> 0 0 0; origin xyz=0.225 0 0.028 rpy=0 0 0 -> xyz=0.24313 -0.012189 -0.023499 rpy=0 0 0
- joint rf_joint1: limit lower=-4 upper=4 effort=20 velocity=16 -> lower=-3 upper=3 effort=20 velocity=16
- joint rf_joint2: limit lower=-4 upper=4 effort=20 velocity=16 -> lower=-3 upper=3 effort=20 velocity=16; origin xyz=0 -0.029287 0.059987 rpy=1.5708 0.0 0 -> xyz=-0.0010387 -0.029268 0.059987 rpy=1.5708 0 0
- joint rf_joint3: limit lower=-4 upper=4 effort=20 velocity=16 -> lower=-3 upper=3 effort=20 velocity=16; origin xyz=0.22999 1.0192E-05 0.0935 rpy=0 0 1.570796325 -> xyz=0.22999 1.0169E-05 0.0935 rpy=0.0 0.0 1.5708
- joint rf_joint4: axis 0 0 1 -> 0 0 0; origin xyz=0.225 0 0.028 rpy=0 0 0 -> xyz=0.24313 -0.013026 -0.023046 rpy=3.1056 0 0

File: descriptions/at_dog_description/xacro/ros2_control_real.xacro (robot description, xacro)
@@ -125,24 +125,4 @@
 			<state_interface name="effort"/>
 		</joint>
-		<sensor name="imu_main_imu">
-			<state_interface name="orientation.w"/>
-			<state_interface name="orientation.x"/>
-			<state_interface name="orientation.y"/>
-			<state_interface name="orientation.z"/>
-			<state_interface name="angular_velocity.x"/>
-			<state_interface name="angular_velocity.y"/>
-			<state_interface name="angular_velocity.z"/>
-			<state_interface name="linear_acceleration.x"/>
-			<state_interface name="linear_acceleration.y"/>
-			<state_interface name="linear_acceleration.z"/>
-		</sensor>
-		<sensor name="odometer">
-			<state_interface name="position.x"/>
-			<state_interface name="position.y"/>
-			<state_interface name="position.z"/>
-			<state_interface name="velocity.x"/>
-			<state_interface name="velocity.y"/>
-			<state_interface name="velocity.z"/>
-		</sensor>
 	</ros2_control>
 </robot>

File: descriptions/at_dog_description/xacro/ros2_control_sim.xacro (robot description, xacro)
@@ -77,24 +77,4 @@
             <state_interface name="effort" />
         </joint>
-        <sensor name="imu_main_imu">
-            <state_interface name="orientation.w" />
-            <state_interface name="orientation.x" />
-            <state_interface name="orientation.y" />
-            <state_interface name="orientation.z" />
-            <state_interface name="angular_velocity.x" />
-            <state_interface name="angular_velocity.y" />
-            <state_interface name="angular_velocity.z" />
-            <state_interface name="linear_acceleration.x" />
-            <state_interface name="linear_acceleration.y" />
-            <state_interface name="linear_acceleration.z" />
-        </sensor>
-        <sensor name="odometer">
-            <state_interface name="position.x" />
-            <state_interface name="position.y" />
-            <state_interface name="position.z" />
-            <state_interface name="velocity.x" />
-            <state_interface name="velocity.y" />
-            <state_interface name="velocity.z" />
-        </sensor>
     </ros2_control>
 </robot>

Commit message: 修复坐标系错误

File: descriptions/at_dog_description/model/dog.urdf (robot description, URDF)
Before this commit: robot at_dog_description, 17 links, 16 joints
Links:
- removed link body_link
- added link base, mass 4.2135; collision mesh filename=package://at_dog_description/model/body_link.stl; visual mesh filename=package://at_dog_description/model/body_link.stl
Joints:
- joint lb_joint1: parent body_link -> base
- joint lf_joint1: parent body_link -> base
- joint rb_joint1: parent body_link -> base
- joint rf_joint1: parent body_link -> base

File: descriptions/at_dog_description/xacro/robot.xacro (robot description, xacro)
@@ -10,5 +10,5 @@
   </xacro:unless>
   <joint name="imu_main_joint" type="fixed">
-    <parent link="body_link"/>
+    <parent link="base"/>
     <child link="imu_main_link"/>
     <origin rpy="0 0 0" xyz="0 0 0.056203"/>
